File: GOTEK Speaker Circuit - On Board/GOTEK Speaker Circuit - On Board.brd (EAGLE design)
At the start: 22.8 x 22.5 mm, 4 parts, among them T1 2N3904

Commit message: Binglesprat
Parts:
- removed JP1: (no value), pinhead:1X04
- added SG1: F/CM12P, buzzer:F/CM12P
Connections:
- net +5V: now also SG1.+; no longer JP1.1
- net SPK-: now also SG1.-; no longer JP1.4
Routing:
- net SPK-: track 0.00 -> 10.7 mm
- net +5V: track 12.7 -> 20.7 mm
Other:
- board size 22.8 x 22.5 mm -> 33 x 22.5 mm
- board text added: "ACTVIE BUZZER CIRCUIT FOR GOTEK FLOPPY USING FLASHFLOPPY ON-BOARD SPEAKER OPTION BY JKELLOGG BASED ON A DESIGN ON THE FLASHFLOPPY GIT WIKI"
- board text removed: "ACTVIE BUZZER CIRCUIT FOR GOTEK FLOPPY USING FLASHFLOPPY EXTERNAL SPEAKER OPTION BY JKELLOGG BASED ON A DESIGN ON THE FLASHFLOPPY GIT WIKI"
- board text removed: "SPK+"
- board text removed: "SPK-"
Changed lines of the file:
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@@
 <layer number="14" name="Route14" color="22" fill="1" visible="no" active="no"/>
 <layer number="15" name="Route15" color="23" fill="1" visible="no" active="no"/>
-<layer number="16" name="Bottom" color="1" fill="1" visible="no" active="yes"/>
+<layer number="16" name="Bottom" color="1" fill="1" visible="yes" active="yes"/>
 <layer number="17" name="Pads" color="2" fill="1" visible="yes" active="yes"/>
 <layer number="18" name="Vias" color="2" fill="1" visible="yes" active="yes"/>
@@
 <board>
 <plain>
-<wire x1="0" y1="0" x2="22.84" y2="0" width="0" layer="20"/>
-<wire x1="22.84" y1="0" x2="22.84" y2="22.53" width="0" layer="20"/>
-<wire x1="22.84" y1="22.53" x2="0" y2="22.53" width="0" layer="20"/>
+<wire x1="0" y1="0" x2="33" y2="0" width="0" layer="20"/>
+<wire x1="33" y1="0" x2="33" y2="22.53" width="0" layer="20"/>
+<wire x1="33" y1="22.53" x2="0" y2="22.53" width="0" layer="20"/>
 <wire x1="0" y1="22.53" x2="0" y2="0" width="0" layer="20"/>
 <text x="5.08" y="2.54" size="1.016" layer="21" align="center-left"> +5V</text>
 <text x="5.08" y="5.08" size="1.016" layer="21" align="center-left"> GND</text>
 <text x="5.08" y="7.62" size="1.016" layer="21" align="center-left"> JB</text>
-<text x="17.78" y="10.16" size="1.016" layer="21" align="center-left"> SPK+</text>
-<text x="17.78" y="2.54" size="1.016" layer="21" align="center-left"> SPK-</text>
-<text x="10.16" y="11.43" size="1.016" layer="22" rot="MR90" align="center">ACTVIE BUZZER CIRCUIT
+<text x="12.7" y="11.43" size="1.016" layer="22" rot="MR270" align="center">ACTVIE BUZZER CIRCUIT
 FOR GOTEK FLOPPY
 USING FLASHFLOPPY
-EXTERNAL SPEAKER OPTION
+ON-BOARD SPEAKER
+OPTION
 BY JKELLOGG
 BASED ON A DESIGN ON
@@
 <attribute name="VALUE" x="8.255" y="11.43" size="1.27" layer="21" ratio="10"/>
 </element>
-<element name="JP1" library="pinhead" library_urn="urn:adsk.eagle:library:325" package="1X04" package3d_urn="urn:adsk.eagle:package:22407/2" value="" x="16.51" y="6.35" smashed="yes" rot="R90">
-<attribute name="NAME" x="14.6812" y="1.1938" size="1.27" layer="25" ratio="10" rot="R90"/>
-<attribute name="POPULARITY" value="91" x="16.51" y="6.35" size="1.778" layer="27" rot="R90" display="off"/>
-<attribute name="VALUE" x="19.685" y="1.27" size="1.27" layer="27" rot="R90"/>
+<element name="SG1" library="buzzer" library_urn="urn:adsk.eagle:library:113" package="F/CM12P" package3d_urn="urn:adsk.eagle:package:5265/1" value="F/CM12P" x="22.86" y="10.16" smashed="yes" rot="R270">
+<attribute name="MF" value="" x="22.86" y="10.16" size="1.778" layer="27" rot="R270" display="off"/>
+<attribute name="MPN" value="" x="22.86" y="10.16" size="1.778" layer="27" rot="R270" display="off"/>
+<attribute name="NAME" x="29.845" y="7.62" size="1.27" layer="25" ratio="10" rot="R270"/>
+<attribute name="OC_FARNELL" value="unknown" x="22.86" y="10.16" size="1.778" layer="27" rot="R270" display="off"/>
+<attribute name="OC_NEWARK" value="unknown" x="22.86" y="10.16" size="1.778" layer="27" rot="R270" display="off"/>
+<attribute name="POPULARITY" value="9" x="22.86" y="10.16" size="1.778" layer="27" rot="R270" display="off"/>
+<attribute name="VALUE" x="19.05" y="14.605" size="1.27" layer="27" ratio="10" rot="R270"/>
 </element>
 </elements>
@@
 <signal name="+5V">
 <contactref element="JP2" pad="1"/>
-<wire x1="16.4592" y1="2.5908" x2="3.81" y2="2.5908" width="0.1524" layer="1"/>
+<contactref element="SG1" pad="+"/>
+<wire x1="19.2024" y1="2.5908" x2="3.81" y2="2.5908" width="0.1524" layer="1"/>
+<wire x1="22.86" y1="6.2484" x2="19.2024" y2="2.5908" width="0.1524" layer="1"/>
 <wire x1="3.81" y1="2.5908" x2="3.81" y2="2.54" width="0.1524" layer="1"/>
-<contactref element="JP1" pad="1"/>
-<wire x1="16.51" y1="2.54" x2="3.81" y2="2.54" width="0" layer="19" extent="1-1"/>
+<wire x1="22.86" y1="6.2484" x2="22.86" y2="6.35" width="0.1524" layer="1"/>
 </signal>
 <signal name="GND">
@@
 <polygon width="0.1524" layer="16">
 <vertex x="0" y="0"/>
-<vertex x="22.86" y="0"/>
-<vertex x="22.86" y="22.86"/>
+<vertex x="33.02" y="0"/>
+<vertex x="33.02" y="22.86"/>
 <vertex x="0" y="22.86"/>
 </polygon>
@@
 <contactref element="T1" pad="2"/>
 <contactref element="R1" pad="2"/>
-<wire x1="5.6388" y1="17.2212" x2="11.43" y2="17.2212" width="0.1524" layer="1"/>
-<wire x1="3.81" y1="19.05" x2="5.6388" y2="17.2212" width="0.1524" layer="1"/>
+<wire x1="9.6012" y1="19.05" x2="3.81" y2="19.05" width="0.1524" layer="1"/>
+<wire x1="11.43" y1="17.2212" x2="9.6012" y2="19.05" width="0.1524" layer="1"/>
 <wire x1="11.43" y1="17.2212" x2="11.43" y2="17.145" width="0.1524" layer="1"/>
 </signal>
@@
 </signal>
 <signal name="SPK-">
-<contactref element="JP1" pad="4"/>
 <contactref element="T1" pad="1"/>
-<wire x1="16.51" y1="10.16" x2="12.7" y2="15.24" width="0" layer="19" extent="1-1"/>
+<contactref element="SG1" pad="-"/>
+<wire x1="21.6408" y1="15.24" x2="12.7" y2="15.24" width="0.1524" layer="1"/>
+<wire x1="22.86" y1="14.0208" x2="21.6408" y2="15.24" width="0.1524" layer="1"/>
+<wire x1="22.86" y1="14.0208" x2="22.86" y2="13.97" width="0.1524" layer="1"/>
 </signal>
 </signals>
