File: C64 ROM Selector - ATTiny85/C64 Rom Selector - ATTiny85.brd (EAGLE design)
At the start: 62.2 x 63.5 mm, 6 parts, among them IC1 C64 ROM SOCKET, IC2 27256 EEPROM, J1 C64, J2 PLED, U1 ATTINY85

Commit message: Updated schematic to clarify pins
Connections:
- net PIN1 renamed RESTORE
- net PIN2 renamed RESET
- net PIN3 renamed EXROM
- net PIN4 renamed PLED
Changed lines of the file:
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@@
 <wire x1="5.08" y1="19.05" x2="5.08" y2="3.81" width="0" layer="19" extent="1-1"/>
 </signal>
-<signal name="PIN1">
+<signal name="RESTORE">
 <contactref element="J1" pad="1"/>
 <contactref element="U1" pad="5"/>
@@
 <wire x1="55.7784" y1="6.2484" x2="55.88" y2="6.35" width="0.1524" layer="1"/>
 </signal>
-<signal name="PIN4">
+<signal name="PLED">
 <contactref element="R2" pad="2"/>
 <contactref element="U1" pad="2"/>
@@
 <wire x1="41.91" y1="10.8204" x2="42.037" y2="10.795" width="0.1524" layer="1"/>
 </signal>
-<signal name="PIN2">
+<signal name="RESET">
 <contactref element="J1" pad="2"/>
 <contactref element="U1" pad="6"/>
@@
 <wire x1="55.7784" y1="8.9916" x2="55.88" y2="8.89" width="0.1524" layer="1"/>
 </signal>
-<signal name="PIN3">
+<signal name="EXROM">
 <contactref element="J1" pad="3"/>
 <contactref element="U1" pad="7"/>
