File: C64 Breakout Boards/Expansion Port.sch (EAGLE design)
At the start: 0 parts

Commit message: Working on Breakouts
Parts:
- added X1, X2: 87758-4416, con-molex:87758-4416
Connections:
- new net N$1: X1-1.S, X2-1.S
- new net N$10: X1-19.S, X2-19.S
- new net N$11: X1-21.S, X2-21.S
- new net N$12: X1-23.S, X2-23.S
- new net N$13: X1-25.S, X2-25.S
- new net N$14: X1-27.S, X2-27.S
- new net N$15: X1-29.S, X2-29.S
- new net N$16: X1-31.S, X2-31.S
- new net N$17: X1-33.S, X2-33.S
- new net N$18: X1-35.S, X2-35.S
- new net N$19: X1-37.S, X2-37.S
- new net N$2: X1-3.S, X2-3.S
- new net N$20: X1-39.S, X2-39.S
- new net N$21: X1-41.S, X2-41.S
- new net N$22: X1-43.S, X2-43.S
- new net N$23: X1-2.S, X2-2.S
- new net N$24: X1-4.S, X2-4.S
- new net N$25: X1-6.S, X2-6.S
- new net N$26: X1-8.S, X2-8.S
- new net N$27: X1-10.S, X2-10.S
- new net N$28: X1-12.S, X2-12.S
- new net N$29: X1-14.S, X2-14.S
- new net N$3: X1-5.S, X2-5.S
- new net N$30: X1-16.S, X2-16.S
- new net N$31: X1-18.S, X2-18.S
- new net N$32: X1-20.S, X2-20.S
- new net N$33: X1-22.S, X2-22.S
- new net N$34: X1-24.S, X2-24.S
- new net N$35: X1-26.S, X2-26.S
- new net N$36: X1-28.S, X2-28.S
- new net N$37: X1-30.S, X2-30.S
- new net N$38: X1-32.S, X2-32.S
- new net N$39: X1-34.S, X2-34.S
- new net N$4: X1-7.S, X2-7.S
- new net N$40: X1-36.S, X2-36.S
- new net N$41: X1-38.S, X2-38.S
- new net N$42: X1-40.S, X2-40.S
- new net N$43: X1-42.S, X2-42.S
- new net N$44: X1-44.S, X2-44.S
- new net N$5: X1-9.S, X2-9.S
- new net N$6: X1-11.S, X2-11.S
- new net N$7: X1-13.S, X2-13.S
- new net N$8: X1-15.S, X2-15.S
- new net N$9: X1-17.S, X2-17.S
